File: Motor Driver Board/Motor Driver Board.kicad_sch (KiCad schematic)
At the start: 29 parts, among them J1 Conn_02x05_Odd_Even, J2 Conn_01x02, J3 Conn_01x04, U1 STSPIN32G4

Commit message: updated pcb
Parts:
- added C14: 220 nF 100V, Capacitor_SMD:C_1206_3216Metric, symbol Device:C
- added C23, C24: 10pF, Capacitor_SMD:C_0603_1608Metric, symbol Device:C
- added JP3: Jumper_2_Open, Connector_PinHeader_2.54mm:PinHeader_1x02_P2.54mm_Vertical, symbol Jumper:Jumper_2_Open
- added R26: 10k, Resistor_SMD:R_0805_2012Metric, symbol Device:R_US
- added Y1: 24.000MHz, Crystal:Crystal_SMD_SeikoEpson_FA128-4Pin_2.0x1.6mm, symbol Device:Crystal_GND24
- C1: footprint (none) -> Capacitor_SMD:C_0603_1608Metric; LCSC (none) -> C1614
- C10, C12, C13, C8: footprint (none) -> Capacitor_SMD:C_0402_1005Metric; LCSC (none) -> C1525
- C11, C9: footprint (none) -> Capacitor_SMD:C_0603_1608Metric; LCSC (none) -> C5673
- C15: footprint (none) -> Capacitor_SMD:C_0603_1608Metric; now not fitted
- C19: footprint Connector:BJB_Pico_46.110.1001_Receptacle_Horizontal -> Capacitor_SMD:C_0805_2012Metric; LCSC (none) -> C15850
- C2, C3, C4: footprint (none) -> Motor Driver Board:CAP-SMD_BD16.0-L17.0-W17.0-FD; LCSC (none) -> C249883
- C7: footprint (none) -> Capacitor_SMD:C_0805_2012Metric; LCSC (none) -> C15850
- D1: footprint (none) -> Diode_SMD:D_SOD-523; LCSC (none) -> C2926449
- D10: footprint (none) -> Diode_SMD:D_SMA; LCSC (none) -> C165701
- J1: footprint (none) -> Connector_PinHeader_2.54mm:PinHeader_2x05_P2.54mm_Vertical; now not fitted
- J2: footprint (none) -> Connector_PinHeader_2.54mm:PinHeader_1x02_P2.54mm_Vertical; now not fitted
- J3: footprint (none) -> Connector_PinHeader_2.54mm:PinHeader_1x04_P2.54mm_Vertical; now not fitted
- L2: footprint (none) -> Motor Driver Board:IND-SMD_L5.0-W5.0_FNR50XXS; LCSC (none) -> C167940
- R10, R7, R8, R9: footprint (none) -> Resistor_SMD:R_0805_2012Metric; LCSC (none) -> C17477
- R11: footprint (none) -> Resistor_SMD:R_0805_2012Metric; LCSC (none) -> C17560
- R12: footprint (none) -> Resistor_SMD:R_0805_2012Metric; LCSC (none) -> C17414
- R19: value 72.3k 1% -> 75k 1%; footprint (none) -> Resistor_SMD:R_0603_1608Metric; LCSC (none) -> C23242
- R20: footprint (none) -> Resistor_SMD:R_0603_1608Metric; LCSC (none) -> C22991
- TP1: footprint (none) -> TestPoint:TestPoint_Pad_D1.5mm; now not fitted
- U1: footprint QFN_IN32G4_STM -> Motor Driver Board:VFQFPN-64_L9.0-W9.0-P0.50-TL-EP4.0; LCSC (none) -> C7434864
Connections:
- net GND: now also C14.2, C23.2, C24.2, R26.2, Y1.2 (G), Y1.4 (G)
- net PA11: now also U1.48 (PA12); no longer U1.47 (PA11)
- net PA12: now also U1.47 (PA11); no longer U1.48 (PA12)
- net VDD: now also JP3.2 (B)
- net VDDA: now also U1.27 (VDDA)
- net VM: now also C14.1
- net VREF+: now also U1.26 (VREF+)
- net VSHUNT1P: now reaches U1.14 (PA1)
- net PA4: now reaches U1.17 (PA4)
- net PA5: now reaches U1.18 (PA5)
- net VSHUNT2P: now reaches U1.20 (PA7)
- net VSHUNT3P: now reaches U1.23 (PB0)
- net PB5: now reaches U1.55 (PB4)
- net PB4: now reaches U1.56 (PB5)
- net at U1.59 (PB8): now also JP3.1 (A), R26.1
- net PF0: now reaches U1.6 (PF0)
- net PF0: now also C24.1, Y1.1
- net PF1: now reaches U1.7 (PF1)
- net PF1: now also C23.1, Y1.3
- no-connect marks 1 -> 23
