File: Motor Driver Board/motor_driver.kicad_sch (KiCad schematic)
At the start: 35 parts, among them Q10 Q_NMOS_GDSD, Q11 Q_NMOS_GDSD, Q12 Q_NMOS_GDSD, Q7 Q_NMOS_GDSD, Q8 Q_NMOS_GDSD, Q9 Q_NMOS_GDSD

Commit message: updated pcb
Parts:
- added J6: Screw_Terminal_01x03, TerminalBlock_MetzConnect:TerminalBlock_MetzConnect_Type073_RT02603HBLU_1x03_P5.08mm_Horizontal, symbol Connector:Screw_Terminal_01x03
- C16, C18, C21: footprint (none) -> Capacitor_SMD:C_0603_1608Metric; LCSC (none) -> C5673
- C17, C20, C22: footprint (none) -> Capacitor_SMD:C_1206_3216Metric; LCSC (none) -> C106047
- D11, D12, D13, D14, D8, D9: LCSC (none) -> C2935154
- JP1, JP2: footprint (none) -> Connector_PinHeader_2.54mm:PinHeader_1x02_P2.54mm_Vertical; now not fitted
- NT1, NT2, NT3: footprint (none) -> NetTie:NetTie-3_SMD_Pad0.5mm
- Q10, Q11, Q12, Q7, Q8, Q9: footprint (none) -> Motor Driver Board:MCAC60N10Y_DFN5060_GDSD; LCSC (none) -> C3277744
- R1, R2, R3, R4, R5, R6: value 100m 1% .5W -> 200m 1% .5W; footprint (none) -> Resistor_SMD:R_1206_3216Metric; LCSC (none) -> C160920
- R13, R14, R15, R16, R17, R18: footprint (none) -> Resistor_SMD:R_0805_2012Metric; LCSC (none) -> C17634
Connections:
- net OUT1: now also J6.1 (Pin_1)
- net OUT2: now also J6.2 (Pin_2)
- net OUT3: now also J6.3 (Pin_3)
