File: Motor Driver Board/Motor Driver Board.kicad_pcb (KiCad board)
At the start: 2 copper layers, 81 parts, among them J1 Conn_02x05_Odd_Even, J2 Conn_01x02, J3 Conn_01x04, J4 Conn_01x03, J5 Conn_01x08, J6 Screw_Terminal_01x03, Q10 Q_NMOS_GDSD, Q11 Q_NMOS_GDSD, Q12 Q_NMOS_GDSD, Q7 Q_NMOS_GDSD, Q8 Q_NMOS_GDSD, Q9 Q_NMOS_GDSD, U1 STSPIN32G4, U2 SN65HVD230, Y1 24.000MHz

Commit message: board schematic finished
Parts:
- added REF**: MountingHole_3.2mm_M3, MountingHole:MountingHole_3.2mm_M3, F.Cu at (88.0, 26.0)
- added REF**: MountingHole_3.2mm_M3, MountingHole:MountingHole_3.2mm_M3, F.Cu at (87.5, 119.0)
- added REF**: MountingHole_3.2mm_M3, MountingHole:MountingHole_3.2mm_M3, F.Cu at (164.5, 119.0)
- added REF**: MountingHole_3.2mm_M3, MountingHole:MountingHole_3.2mm_M3, F.Cu at (165.0, 25.5)
- moved C4 98.2 mm to (142.0, 36.5), turned to 90 degrees
- moved TP1 91.9 mm to (135.0, 110.0)
- moved J6 82.8 mm to (151.4, 63.1), turned to 90 degrees
- moved C3 73.9 mm to (123.7, 36.5), turned to 90 degrees
- moved R10 71.1 mm to (133.5, 103.4), turned to 90 degrees
- moved R22 67.4 mm to (145.0, 96.8), turned to -90 degrees
- moved R8 65.2 mm to (117.5, 103.2), turned to -90 degrees
- moved R9 63.8 mm to (127.5, 96.2), turned to 90 degrees
- moved R21 62.5 mm to (139.9, 92.8), turned to 180 degrees
- moved R7 62.1 mm to (115.0, 98.2), turned to -90 degrees
- moved R23 59.7 mm to (112.0, 101.2), turned to 180 degrees
- moved R18 58.9 mm to (142.5, 75.9), turned to 90 degrees
- moved J4 58.5 mm to (134.0, 99.2), turned to 180 degrees
- moved U2 57.5 mm to (140.0, 96.8)
- moved R17 56.7 mm to (139.0, 75.9), turned to 90 degrees
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Routing:
- net VM: track 0.00 -> 95.4 mm
- net OUT1: track 0.00 -> 55.8 mm
- net OUT3: track 0.00 -> 55.0 mm, vias 0 -> 1
- net OUT2: track 0.00 -> 21.2 mm
- net /Motor Driver/VSHUNT2P: track 0.00 -> 5.09 mm
- net /Motor Driver/VSHUNT1P: track 0.00 -> 4.73 mm
- net /Motor Driver/VSHUNT3P: track 0.00 -> 4.21 mm
Other:
- board outline added: 87 x 103.5 mm
- copper layers 2 -> 4

Commit message: board routed
Parts:
- moved C22 87.3 mm to (152.3, 30.8), turned to 90 degrees
- moved C20 76.5 mm to (135.0, 33.4), turned to 90 degrees
- moved JP1 66.5 mm to (142.0, 59.6), turned to -90 degrees
- moved JP2 57.6 mm to (121.9, 59.9), turned to -90 degrees
- moved C14 51.6 mm to (118.8, 97.8)
- moved D11 50.8 mm to (160.0, 38.9), turned to 180 degrees
- moved R15 50.4 mm to (160.3, 36.1), turned to 180 degrees
- moved J2 49.1 mm to (127.5, 120.2), turned to 90 degrees
- moved C4 47.3 mm to (94.9, 40.8), turned to 180 degrees
- moved J1 44.9 mm to (117.3, 69.3), turned to -90 degrees
- moved TP1 43.3 mm to (93.0, 120.6)
- moved C2 42.2 mm to (94.9, 77.4), turned to 180 degrees
- moved D13 41.0 mm to (145.1, 36.5), turned to 180 degrees
- moved D8 37.7 mm to (122.3, 36.8), turned to 180 degrees
- moved R17 37.3 mm to (144.7, 39.0), turned to 180 degrees
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Routing:
- net VDD: track 0.00 -> 153.2 mm, vias 0 -> 12
- net GHS1: track 0.00 -> 118.0 mm, vias 0 -> 6
- net GHS2: track 0.00 -> 90.0 mm, vias 0 -> 6
- net VM: track 95.4 -> 172.5 mm, vias 0 -> 7
- net /Root/SCREF: track 0.00 -> 75.7 mm, vias 0 -> 5
- net GHS3: track 0.00 -> 73.8 mm, vias 0 -> 4
- net OUT3: track 55.0 -> 127.9 mm, vias 1 -> 6
- net OUT2: track 21.2 -> 86.4 mm
- net Net-(JP3-A): track 0.00 -> 64.6 mm, vias 0 -> 3
- net PA4: track 0.00 -> 63.6 mm, vias 0 -> 4
- net GLS1: track 0.00 -> 61.7 mm
- net PA11: track 0.00 -> 61.0 mm, vias 0 -> 6
- net /Root/PG10: track 0.00 -> 60.5 mm, vias 0 -> 2
- net Net-(J5-Pin_3): track 0.00 -> 60.2 mm, vias 0 -> 4
- net GLS3: track 0.00 -> 48.8 mm, vias 0 -> 2
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